File: generative_picture_hardware.kicad_sch (KiCad schematic)
At the start: 0 parts

Commit message: Start the schematics by connecting the HAT pins to the ESP32
The VCC on the e-Paper HAT is connected to 5V[1], but we will power it from
the 3V3 rails as I did in all my tests*. Because of that, we can't
replicate the pinout of the raspberry Pi header exactly. Instead, we
connect 3V3 to where 5V is on the Pi and leave the pins where the Pi has
3V3 unconnected (even though they're not routed in the HAT).

* The level shifter in the HAT (a TXS0108E[2]) takes from 1.65 to 5.5V on the
B port, where VCC is routed.

[1]: https://www.waveshare.com/w/upload/8/87/E-Paper-Driver-HAT-Schematic.pdf
[2]: https://www.ti.com/lit/ds/symlink/txs0108e.pdf?ts=1611473568779
Parts:
- added C?: C_Small, symbol Device:C_Small
- added J?: e_Paper_HAT, symbol Connector_Generic:Conn_02x20_Odd_Even
- added U?: ESP32-WROOM-32, RF_Module:ESP32-WROOM-32, symbol RF_Module:ESP32-WROOM-32
Connections:
- new net: U?.1 (GND), U?.15 (GND), U?.38 (GND), U?.39 (GND)
- new net +3V3: C?.1, J?.2 (Pin_2), J?.4 (Pin_4)
- new net EPD_BUSY: J?.18 (Pin_18), U?.26 (IO4)
- new net EPD_CLK: J?.23 (Pin_23), U?.30 (IO18)
- new net EPD_CS: J?.24 (Pin_24), U?.29 (IO5)
- new net EPD_DC: J?.22 (Pin_22), U?.28 (IO17)
- new net EPD_MOSI: J?.19 (Pin_19), U?.37 (IO23)
- new net EPD_RST: J?.11 (Pin_11), U?.27 (IO16)
- new net GND: C?.2, J?.14 (Pin_14), J?.20 (Pin_20), J?.25 (Pin_25), J?.30 (Pin_30), J?.34 (Pin_34), J?.39 (Pin_39), J?.6 (Pin_6), J?.9 (Pin_9)
- no-connect marks 0 -> 24
Other:
- note added: "Note: Pins 2 and 4 on the RPi are 5V. On the E-Paper HAT from waveshare VCC is connected to 5V, but since we're going to power it from 3V3, we need to switch out in our connector. To avoid any issues, we leave the RPi's 3V3 (pins 1 and 17) unconnected (even though they're not routed in the HAT)."
- note added: "Power"
- note added: "e-Paper HAT connector"
- note added: "µC"
